File: Paint Perfector.kicad_sch (KiCad schematic)
At the start: 13 parts, among them J1 Power, J2 Digital/PWM, J3 Analog, J4 Digital/PWM, SW1 Pushbutton, SW2 Pushbutton, SW3 Pushbutton, SW4 Pushbutton

Commit message: Newst one
Parts:
- added H1, H2, H3: Motor Controller, symbol Auxiliary_Items:Generic_Outline
- added H4: MixerMotor Controller, symbol Auxiliary_Items:Generic_Outline
- added J5: Power, Connector_PinSocket_2.54mm:PinSocket_1x08_P2.54mm_Vertical, symbol Connector_Generic:Conn_01x08
- added J6: Analog, Connector_PinSocket_2.54mm:PinSocket_1x06_P2.54mm_Vertical, symbol Connector_Generic:Conn_01x06
- added J7: Digital/PWM, Connector_PinSocket_2.54mm:PinSocket_1x10_P2.54mm_Vertical, symbol Connector_Generic:Conn_01x10
- added J8: Digital/PWM, Connector_PinSocket_2.54mm:PinSocket_1x08_P2.54mm_Vertical, symbol Connector_Generic:Conn_01x08
- added SW5: SW_DIP_x01, symbol Switch:SW_DIP_x01
Connections:
- net *10: now also J7.8 (Pin_8)
- net *11: now also J7.7 (Pin_7)
- net *3: now also J8.5 (Pin_5)
- net *5: now also J8.3 (Pin_3)
- net *6: now also J8.2 (Pin_2)
- net +6V: now also SW5.2
- net 2: now also J8.6 (Pin_6)
- net 4: now also J8.4 (Pin_4)
- net 7: now also J8.1 (Pin_1)
- net AREF: now also J7.3 (Pin_3)
- net GND: now also J5.6 (Pin_6), J5.7 (Pin_7), J7.4 (Pin_4)
- net IOREF: now also J5.2 (Pin_2)
- net RX/0: now also J8.8 (Pin_8)
- net SCL/A5: now also J6.6 (Pin_6), J7.1 (Pin_1)
- net SDA/A4: now also J6.5 (Pin_5), J7.2 (Pin_2)
- net TX/1: now also J8.7 (Pin_7)
- net ~{RESET}: now also J5.3 (Pin_3)
- no-connect marks 1 -> 2
